File: AP.sch (KiCad schematic (older format))
At the start: 16 parts, among them J1 Conn_01x06_Female, J2 Conn_01x01_Female, J3 Conn_01x02_Female, J4 Conn_01x03_Female, J5 Conn_01x01_Female, J6 Conn_01x04_Female, U1 74HC04, U2 DS3231MZ, U3 74HC04, U4 74HC04, U5 74HC04

Commit message: Update AP.sch
Parts:
- removed J1: Conn_01x06_Female, Connector_PinHeader_2.54mm:PinHeader_1x06_P2.54mm_Vertical, symbol Connector:Conn_01x06_Female
- removed J2, J5: Conn_01x01_Female, Connector_PinHeader_2.54mm:PinHeader_1x01_P2.54mm_Vertical, symbol Connector:Conn_01x01_Female
- removed J3: Conn_01x02_Female, Connector_PinHeader_2.54mm:PinHeader_1x02_P2.54mm_Vertical, symbol Connector:Conn_01x02_Female
- removed J4: Conn_01x03_Female, Connector_PinHeader_2.54mm:PinHeader_1x03_P2.54mm_Vertical, symbol Connector:Conn_01x03_Female
- removed J6: Conn_01x04_Female, Connector_PinHeader_2.54mm:PinHeader_1x04_P2.54mm_Vertical, symbol Connector:Conn_01x04_Female
- removed R1: RTRIM, Potentiometer_THT:Potentiometer_ACP_CA6-H2,5_Horizontal, symbol Device:RTRIM
- added Analogin: Conn_01x06_Male, symbol Connector:Conn_01x06_Male
- added Baterie: Battery_Cell, symbol Device:Battery_Cell
- added Digital1, Power: Conn_01x08_Male, symbol Connector:Conn_01x08_Male
- added Digital2: Conn_01x10_Male, symbol Connector:Conn_01x10_Male
- added Rtrim: R_POT, symbol Device:R_POT
- added tlačítko1, tlačítko2: SW_MEC_5G, symbol Switch:SW_MEC_5G
- R: renamed from R2; value R -> 220
- R: renamed from R3; value R -> 220
- R: renamed from R4; value R -> 220
- R: renamed from R5; value R -> 220
- renumbered U4 to Demultiplexor, U5 to Displej, U1 to I1, U1 to I3, U1 to I4, U1 to I5, U1 to I6, U1 to Inv1, U3 to Inv2, U3 to Inv21, U3 to Inv22, U2 to RTC
Connections:
- net labels added: A0, A1, A2, GNDs12, GNDs6, GNDs8, GNDs9, Rtrim1, SCL, SDA, Tl1, Tl2, Y0, Y1, Y2, Y3, Y4, Y5, Y6, Y7
- wire segments 105 -> 88
- no-connect marks 0 -> 21
Other:
- note added: "Demultiplexor\n"
- note added: "Invertory a 7seg\n"
- note added: "Piny procesor\n"
- note added: "RTC"
- note added: "trimer a tlačítko\n"
- moved on the sheet: Demultiplexor, Displej, I1A, I3B, I4D, I5E, I6F, Inv1G, Inv21A, Inv22B, Inv2G, R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

Commit message: Update AP.sch
Parts:
- added C1: 10nF, symbol Device:CP
- added C2: 1nF, symbol Device:CP
- added RI2c, RI2c1: R, symbol Device:R
- added Rtl1, Rtl2: 4k3, symbol Device:R
- Demultiplexor: value 74HC04 -> 74HC138
- Displej: value 74HC04 -> Disp
Connections:
- net GND: now also C1.2, C2.2, Rtl1.2, Rtl2.2
- net SCL: now also RI2c1.2
- net SDA: now also RI2c.2
- net Tl1: now also Rtl1.1
- net Tl2: now also Rtl2.1
- net VCC: now also C1.1, C2.1, RI2c.1, RI2c1.1
Other:
- moved on the sheet: Baterie, RTC

Commit message: Update AP.sch
Parts:
- RI2c, RI2c1: value R -> 4k7
- Rtl1, Rtl2: value 4k3 -> 10k
Changed lines of the file:
@@
 Text Notes 2500 700  0    118  ~ 0
 Demultiplexor\n
-$Comp
-L power:VCC #PWR0104
-U 1 1 60044EB4
-P 4400 900
-F 0 "#PWR0104" H 4400 750 50  0001 C CNN
-F 1 "VCC" V 4415 1027 50  0000 L CNN
-F 2 "" H 4400 900 50  0001 C CNN
-F 3 "" H 4400 900 50  0001 C CNN
-	1    4400 900
-	0    -1   -1   0
-$EndComp
-$Comp
-L power:GND #PWR0105
-U 1 1 600469CE
-P 5800 900
-F 0 "#PWR0105" H 5800 650 50  0001 C CNN
-F 1 "GND" V 5805 772 50  0000 R CNN
-F 2 "" H 5800 900 50  0001 C CNN
-F 3 "" H 5800 900 50  0001 C CNN
-	1    5800 900
-	0    -1   -1   0
-$EndComp
-Wire Wire Line
-	5600 900  5800 900
-Wire Wire Line
-	4400 900  4600 900
 Wire Wire Line
 	4750 1350 4500 1350
@@
 Wire Wire Line
 	5350 2850 6375 2850
-$Comp
-L power:GND #PWR0106
-U 1 1 600A584B
-P 5875 3450
-F 0 "#PWR0106" H 5875 3200 50  0001 C CNN
-F 1 "GND" V 5880 3322 50  0000 R CNN
-F 2 "" H 5875 3450 50  0001 C CNN
-F 3 "" H 5875 3450 50  0001 C CNN
-	1    5875 3450
-	0    -1   -1   0
-$EndComp
-$Comp
-L power:VCC #PWR0107
-U 1 1 600A6F71
-P 4325 3450
-F 0 "#PWR0107" H 4325 3300 50  0001 C CNN
-F 1 "VCC" V 4340 3578 50  0000 L CNN
-F 2 "" H 4325 3450 50  0001 C CNN
-F 3 "" H 4325 3450 50  0001 C CNN
-	1    4325 3450
-	0    -1   -1   0
-$EndComp
-Wire Wire Line
-	4625 3450 4325 3450
-Wire Wire Line
-	5875 3450 5625 3450
 Wire Wire Line
 	4750 3925 4500 3925
@@
 Wire Notes Line
 	3750 4625 10900 4625
-Wire Wire Line
-	1250 1000 1025 1000
-Wire Wire Line
-	1250 1150 1025 1150
-$Comp
-L power:GND #PWR?
-U 1 1 6005CA21
-P 1025 1000
-F 0 "#PWR?" H 1025 750 50  0001 C CNN
-F 1 "GND" V 1030 872 50  0000 R CNN
-F 2 "" H 1025 1000 50  0001 C CNN
-F 3 "" H 1025 1000 50  0001 C CNN
-	1    1025 1000
-	0    1    1    0
-$EndComp
-$Comp
-L power:GND #PWR?
-U 1 1 6005DC48
-P 1025 1150
-F 0 "#PWR?" H 1025 900 50  0001 C CNN
-F 1 "GND" V 1030 1022 50  0000 R CNN
-F 2 "" H 1025 1150 50  0001 C CNN
-F 3 "" H 1025 1150 50  0001 C CNN
-	1    1025 1150
-	0    1    1    0
-$EndComp
-Wire Wire Line
-	1250 1300 1025 1300
-$Comp
-L power:VCC #PWR?
-U 1 1 60062081
-P 1025 1300
-F 0 "#PWR?" H 1025 1150 50  0001 C CNN
-F 1 "VCC" V 1040 1427 50  0000 L CNN
-F 2 "" H 1025 1300 50  0001 C CNN
-F 3 "" H 1025 1300 50  0001 C CNN
-	1    1025 1300
-	0    -1   -1   0
-$EndComp
 NoConn ~ 2075 4800
 NoConn ~ 2075 4900
@@
 P 975 6275
 F 0 "RI2c1" H 1045 6321 50  0000 L CNN
-F 1 "R" H 1045 6230 50  0000 L CNN
+F 1 "4k7" H 1045 6230 50  0000 L CNN
 F 2 "" V 905 6275 50  0001 C CNN
 F 3 "~" H 975 6275 50  0001 C CNN
@@
 P 1225 6275
 F 0 "RI2c" H 1295 6321 50  0000 L CNN
-F 1 "R" H 1295 6230 50  0000 L CNN
+F 1 "4k7" H 1295 6230 50  0000 L CNN
 F 2 "" V 1155 6275 50  0001 C CNN
 F 3 "~" H 1225 6275 50  0001 C CNN
@@
 P 9000 5600
 F 0 "Rtl1" H 9070 5646 50  0000 L CNN
-F 1 "4k3 " H 9070 5555 50  0000 L CNN
+F 1 "10k" H 9070 5555 50  0000 L CNN
 F 2 "" V 8930 5600 50  0001 C CNN
 F 3 "~" H 9000 5600 50  0001 C CNN
@@
 P 10475 5600
 F 0 "Rtl2" H 10545 5646 50  0000 L CNN
-F 1 "4k3" H 10545 5555 50  0000 L CNN
+F 1 "10k" H 10545 5555 50  0000 L CNN
 F 2 "" V 10405 5600 50  0001 C CNN
 F 3 "~" H 10475 5600 50  0001 C CNN
@@
 Wire Wire Line
 	9000 5825 9000 5750
+$Comp
+L power:VCC #PWR?
+U 1 1 5FFFC260
+P 4375 800
+F 0 "#PWR?" H 4375 650 50  0001 C CNN
+F 1 "VCC" H 4390 973 50  0000 C CNN
+F 2 "" H 4375 800 50  0001 C CNN
+F 3 "" H 4375 800 50  0001 C CNN
+	1    4375 800
+	1    0    0    -1
+$EndComp
+Wire Wire Line
+	4375 800  4375 900
+Wire Wire Line
+	4375 900  4600 900
+$Comp
+L power:VCC #PWR?
+U 1 1 60001D36
+P 4375 3375
+F 0 "#PWR?" H 4375 3225 50  0001 C CNN
+F 1 "VCC" H 4390 3548 50  0000 C CNN
+F 2 "" H 4375 3375 50  0001 C CNN
+F 3 "" H 4375 3375 50  0001 C CNN
+	1    4375 3375
+	1    0    0    -1
+$EndComp
+Wire Wire Line
+	4375 3375 4375 3450
+Wire Wire Line
+	4375 3450 4625 3450
+$Comp
+L power:GND #PWR?
+U 1 1 6000776B
+P 5825 975
+F 0 "#PWR?" H 5825 725 50  0001 C CNN
+F 1 "GND" H 5830 802 50  0000 C CNN
+F 2 "" H 5825 975 50  0001 C CNN
+F 3 "" H 5825 975 50  0001 C CNN
+	1    5825 975
+	1    0    0    -1
+$EndComp
+$Comp
+L power:GND #PWR?
+U 1 1 60008B18
+P 5875 3525
+F 0 "#PWR?" H 5875 3275 50  0001 C CNN
+F 1 "GND" H 5880 3352 50  0000 C CNN
+F 2 "" H 5875 3525 50  0001 C CNN
+F 3 "" H 5875 3525 50  0001 C CNN
+	1    5875 3525
+	1    0    0    -1
+$EndComp
+Wire Wire Line
+	5625 3450 5875 3450
+Wire Wire Line
+	5875 3450 5875 3525
+Wire Wire Line
+	5600 900  5825 900
+Wire Wire Line
+	5825 900  5825 975
+$Comp
+L power:VCC #PWR?
+U 1 1 6002B037
+P 1075 850
+F 0 "#PWR?" H 1075 700 50  0001 C CNN
+F 1 "VCC" H 1090 1023 50  0000 C CNN
+F 2 "" H 1075 850 50  0001 C CNN
+F 3 "" H 1075 850 50  0001 C CNN
+	1    1075 850
+	1    0    0    -1
+$EndComp
+Wire Wire Line
+	1250 1300 1075 1300
+Wire Wire Line
+	1075 1300 1075 850
+$Comp
+L power:GND #PWR?
+U 1 1 6003141D
+P 900 1200
+F 0 "#PWR?" H 900 950 50  0001 C CNN
+F 1 "GND" H 905 1027 50  0000 C CNN
+F 2 "" H 900 1200 50  0001 C CNN
+F 3 "" H 900 1200 50  0001 C CNN
+	1    900  1200
+	1    0    0    -1
+$EndComp
+$Comp
+L power:GND #PWR?
+U 1 1 600320D8
+P 675 1000
+F 0 "#PWR?" H 675 750 50  0001 C CNN
+F 1 "GND" H 680 827 50  0000 C CNN
+F 2 "" H 675 1000 50  0001 C CNN
+F 3 "" H 675 1000 50  0001 C CNN
+	1    675  1000
+	1    0    0    -1
+$EndComp
+Wire Wire Line
+	675  1000 1250 1000
+Wire Wire Line
+	1250 1150 900  1150
+Wire Wire Line
+	900  1150 900  1200
 $EndSCHEMATC
