File: AP.sch (KiCad schematic (older format))
At the start: 31 parts, among them U1 74HC04

Commit message: 1
Parts:
- Analogin1: renamed from Analogin; footprint (none) -> Connector_PinHeader_2.54mm:PinHeader_1x06_P2.54mm_Vertical
- Baterie1: renamed from Baterie; footprint (none) -> Battery:BatteryHolder_Keystone_1060_1x2032
- C1, C2: footprint (none) -> Capacitor_SMD:C_0805_2012Metric
- Demultiplexor1: renamed from Demultiplexor; footprint Package_DIP:DIP-16_W7.62mm -> Package_SO:SO-16_3.9x9.9mm_P1.27mm
- Digital1: footprint (none) -> Connector_PinHeader_2.54mm:PinHeader_1x08_P2.54mm_Vertical
- Digital2: footprint (none) -> Connector_PinHeader_2.54mm:PinHeader_1x10_P2.54mm_Vertical
- I1, I3, I4, I5, I6, Inv1, Inv2, Inv21, Inv22, U1: footprint Package_DIP:DIP-14_W7.62mm_Socket -> Package_SO:SO-14_3.9x8.65mm_P1.27mm
- Power1: renamed from Power; footprint (none) -> Connector_PinHeader_2.54mm:PinHeader_1x08_P2.54mm_Vertical
- R1, R2, R3, R4: renamed from R; footprint Resistor_THT:R_Axial_DIN0204_L3.6mm_D1.6mm_P5.08mm_Horizontal -> Resistor_SMD:R_0805_2012Metric
- RI2c1, Rtl1, Rtl2: footprint (none) -> Resistor_SMD:R_0805_2012Metric
- RI2c2: renamed from RI2c; footprint (none) -> Resistor_SMD:R_0805_2012Metric
- RTC1: renamed from RTC; footprint Connector_PinHeader_2.54mm:PinHeader_1x06_P2.54mm_Vertical -> Package_SO:SO-8_3.9x4.9mm_P1.27mm
- renumbered Displej to Displej1, Rtrim to Rtrim1

Commit message: 1
Parts:
- removed Rtl1, Rtl2: 10k, Resistor_SMD:R_0805_2012Metric, symbol Device:R
- removed Rtrim1: R_POT, symbol Device:R_POT
- removed tlačítko1, tlačítko2: SW_MEC_5G, symbol Switch:SW_MEC_5G
- added Nastavení: nastavení hodin, symbol Device:Rotary_Encoder_Switch
- added Rec1, Rec2, Rec3: 10K, symbol Device:R
Connections:
- net labels removed: Rtrim1, Tl1, Tl2
- wire segments 123 -> 124
Other:
- note added: "Ecs\n\n"
- note removed: "trimer a tlačítko\n"
Changed lines of the file:
@@
 Text GLabel 4500 2850 0    50   Input ~ 0
 Y5
-Wire Wire Line
-	7425 5125 7425 5000
-$Comp
-L power:VCC #PWR0108
-U 1 1 5FF8B6C2
-P 7425 5000
-F 0 "#PWR0108" H 7425 4850 50  0001 C CNN
-F 1 "VCC" H 7440 5173 50  0000 C CNN
-F 2 "" H 7425 5000 50  0001 C CNN
-F 3 "" H 7425 5000 50  0001 C CNN
-	1    7425 5000
-	1    0    0    -1
-$EndComp
-Wire Wire Line
-	7425 5425 7425 5600
-$Comp
-L power:GND #PWR0109
-U 1 1 5FF8DBFE
-P 7425 5600
-F 0 "#PWR0109" H 7425 5350 50  0001 C CNN
-F 1 "GND" H 7430 5427 50  0000 C CNN
-F 2 "" H 7425 5600 50  0001 C CNN
-F 3 "" H 7425 5600 50  0001 C CNN
-	1    7425 5600
-	1    0    0    -1
-$EndComp
-$Comp
-L Device:R_POT Rtrim1
-U 1 1 5FF900FB
-P 7425 5275
-F 0 "Rtrim1" H 7356 5321 50  0000 R CNN
-F 1 "R_POT" H 7356 5230 50  0000 R CNN
-F 2 "" H 7425 5275 50  0001 C CNN
-F 3 "~" H 7425 5275 50  0001 C CNN
-	1    7425 5275
-	1    0    0    -1
-$EndComp
-Wire Wire Line
-	7575 5275 7825 5275
-Text GLabel 7825 5275 2    39   Input ~ 0
-Rtrim1
-Wire Wire Line
-	1025 4375 1225 4375
-Text GLabel 1225 4375 2    39   Input ~ 0
-Rtrim1
-$Comp
-L Switch:SW_MEC_5G tlačítko1
-U 1 1 5FFA02FD
-P 8700 5300
-F 0 "tlačítko1" H 8700 5585 50  0000 C CNN
-F 1 "SW_MEC_5G" H 8700 5494 50  0000 C CNN
-F 2 "" H 8700 5500 50  0001 C CNN
-F 3 "http://www.apem.com/int/index.php?controller=attachment&id_attachment=488" H 8700 5500 50  0001 C CNN
-	1    8700 5300
-	1    0    0    -1
-$EndComp
 Wire Notes Line
 	6975 4625 6975 6550
 Wire Notes Line
 	10900 6550 10900 4625
-Text Notes 10775 4800 2    118  ~ 0
-trimer a tlačítko\n
-Wire Wire Line
-	8500 5300 8350 5300
-$Comp
-L power:VCC #PWR0104
-U 1 1 5FFAF2E9
-P 8350 5150
-F 0 "#PWR0104" H 8350 5000 50  0001 C CNN
-F 1 "VCC" H 8365 5323 50  0000 C CNN
-F 2 "" H 8350 5150 50  0001 C CNN
-F 3 "" H 8350 5150 50  0001 C CNN
-	1    8350 5150
-	1    0    0    -1
-$EndComp
-Wire Wire Line
-	8900 5300 9000 5300
-Text GLabel 9075 5300 2    39   Input ~ 0
-Tl1
-Wire Wire Line
-	1025 4475 1225 4475
-Text GLabel 1225 4475 2    39   Input ~ 0
-Tl1
-Wire Wire Line
-	1025 4575 1225 4575
-Text GLabel 1225 4575 2    39   Input ~ 0
-Tl2
-$Comp
-L Switch:SW_MEC_5G tlačítko2
-U 1 1 5FFB9FEB
-P 10150 5300
-F 0 "tlačítko2" H 10150 5585 50  0000 C CNN
-F 1 "SW_MEC_5G" H 10150 5494 50  0000 C CNN
-F 2 "" H 10150 5500 50  0001 C CNN
-F 3 "http://www.apem.com/int/index.php?controller=attachment&id_attachment=488" H 10150 5500 50  0001 C CNN
-	1    10150 5300
-	1    0    0    -1
-$EndComp
-Wire Wire Line
-	9950 5300 9750 5300
-Wire Wire Line
-	10350 5300 10475 5300
-$Comp
-L power:VCC #PWR0105
-U 1 1 5FFBF697
-P 9750 5150
-F 0 "#PWR0105" H 9750 5000 50  0001 C CNN
-F 1 "VCC" H 9765 5323 50  0000 C CNN
-F 2 "" H 9750 5150 50  0001 C CNN
-F 3 "" H 9750 5150 50  0001 C CNN
-	1    9750 5150
-	1    0    0    -1
-$EndComp
-Text GLabel 10575 5300 2    39   Input ~ 0
-Tl2
+Text Notes 10825 4975 2    118  ~ 0
+Ecs\n\n
 Wire Wire Line
 	2050 3000 2275 3000
@@
 	3150 6600 3400 6600
 Connection ~ 3150 6600
-Wire Wire Line
-	10475 5300 10475 5450
-Connection ~ 10475 5300
-Wire Wire Line
-	10475 5300 10575 5300
-Wire Wire Line
-	9000 5300 9000 5450
-Connection ~ 9000 5300
-Wire Wire Line
-	9000 5300 9075 5300
-$Comp
-L Device:R Rtl1
-U 1 1 60066593
-P 9000 5600
-F 0 "Rtl1" H 9070 5646 50  0000 L CNN
-F 1 "10k" H 9070 5555 50  0000 L CNN
-F 2 "Resistor_SMD:R_0805_2012Metric" V 8930 5600 50  0001 C CNN
-F 3 "~" H 9000 5600 50  0001 C CNN
-	1    9000 5600
-	1    0    0    -1
-$EndComp
-$Comp
-L Device:R Rtl2
-U 1 1 600673B8
-P 10475 5600
-F 0 "Rtl2" H 10545 5646 50  0000 L CNN
-F 1 "10k" H 10545 5555 50  0000 L CNN
-F 2 "Resistor_SMD:R_0805_2012Metric" V 10405 5600 50  0001 C CNN
-F 3 "~" H 10475 5600 50  0001 C CNN
-	1    10475 5600
-	1    0    0    -1
-$EndComp
-$Comp
-L power:GND #PWR0111
-U 1 1 60067D58
-P 9000 5825
-F 0 "#PWR0111" H 9000 5575 50  0001 C CNN
-F 1 "GND" H 9005 5652 50  0000 C CNN
-F 2 "" H 9000 5825 50  0001 C CNN
-F 3 "" H 9000 5825 50  0001 C CNN
-	1    9000 5825
-	1    0    0    -1
-$EndComp
-$Comp
-L power:GND #PWR0112
-U 1 1 6006DC8F
-P 10475 5825
-F 0 "#PWR0112" H 10475 5575 50  0001 C CNN
-F 1 "GND" H 10480 5652 50  0000 C CNN
-F 2 "" H 10475 5825 50  0001 C CNN
-F 3 "" H 10475 5825 50  0001 C CNN
-	1    10475 5825
-	1    0    0    -1
-$EndComp
-Wire Wire Line
-	10475 5825 10475 5750
-Wire Wire Line
-	9000 5825 9000 5750
 $Comp
 L power:VCC #PWR0113
@@
 	1    0    0    -1
 $EndComp
-Wire Wire Line
-	8350 5300 8350 5150
-Wire Wire Line
-	9750 5300 9750 5150
+$Comp
+L Device:Rotary_Encoder_Switch Nastavení
+U 1 1 60004A19
+P 9125 5725
+F 0 "Nastavení" H 9125 6092 50  0000 C CNN
+F 1 "nastavení hodin" H 9125 6001 50  0000 C CNN
+F 2 "" H 8975 5885 50  0001 C CNN
+F 3 "~" H 9125 5985 50  0001 C CNN
+	1    9125 5725
+	1    0    0    -1
+$EndComp
+$Comp
+L Device:R Rec1
+U 1 1 60019FB4
+P 8475 5175
+F 0 "Rec1" H 8545 5221 50  0000 L CNN
+F 1 "10K" H 8545 5130 50  0000 L CNN
+F 2 "" V 8405 5175 50  0001 C CNN
+F 3 "~" H 8475 5175 50  0001 C CNN
+	1    8475 5175
+	1    0    0    -1
+$EndComp
+$Comp
+L Device:R Rec2
+U 1 1 6001B1FB
+P 8175 5175
+F 0 "Rec2" H 8245 5221 50  0000 L CNN
+F 1 "10K" H 8245 5130 50  0000 L CNN
+F 2 "" V 8105 5175 50  0001 C CNN
+F 3 "~" H 8175 5175 50  0001 C CNN
+	1    8175 5175
+	1    0    0    -1
+$EndComp
+$Comp
+L Device:R Rec3
+U 1 1 6001BC24
+P 7875 5175
+F 0 "Rec3" H 7945 5221 50  0000 L CNN
+F 1 "10K" H 7945 5130 50  0000 L CNN
+F 2 "" V 7805 5175 50  0001 C CNN
+F 3 "~" H 7875 5175 50  0001 C CNN
+	1    7875 5175
+	1    0    0    -1
+$EndComp
+Wire Wire Line
+	9425 5625 9575 5625
+Wire Wire Line
+	9575 5625 9575 5450
+Wire Wire Line
+	9575 5450 8475 5450
+Wire Wire Line
+	8475 5325 8475 5450
+Connection ~ 8475 5450
+Wire Wire Line
+	8475 5450 7725 5450
+Wire Wire Line
+	8825 5825 8175 5825
+Wire Wire Line
+	8175 5325 8175 5825
+Connection ~ 8175 5825
+Wire Wire Line
+	8175 5825 7725 5825
+Wire Wire Line
+	8825 5625 7875 5625
+Wire Wire Line
+	7875 5325 7875 5625
+Connection ~ 7875 5625
+Wire Wire Line
+	7875 5625 7725 5625
+Wire Wire Line
+	8825 5725 8600 5725
+Wire Wire Line
+	8600 5725 8600 6075
+$Comp
+L power:GND #PWR?
+U 1 1 6004F39A
+P 8600 6075
+F 0 "#PWR?" H 8600 5825 50  0001 C CNN
+F 1 "GND" H 8605 5902 50  0000 C CNN
+F 2 "" H 8600 6075 50  0001 C CNN
+F 3 "" H 8600 6075 50  0001 C CNN
+	1    8600 6075
+	1    0    0    -1
+$EndComp
+Wire Wire Line
+	9425 5825 9575 5825
+Wire Wire Line
+	9575 5825 9575 6025
+$Comp
+L power:GND #PWR?
+U 1 1 60054E38
+P 9575 6025
+F 0 "#PWR?" H 9575 5775 50  0001 C CNN
+F 1 "GND" H 9580 5852 50  0000 C CNN
+F 2 "" H 9575 6025 50  0001 C CNN
+F 3 "" H 9575 6025 50  0001 C CNN
+	1    9575 6025
+	1    0    0    -1
+$EndComp
+Wire Wire Line
+	8475 5025 8175 5025
+Wire Wire Line
+	7875 5025 8175 5025
+Connection ~ 8175 5025
+Wire Wire Line
+	7875 5025 7650 5025
+Connection ~ 7875 5025
+$Comp
+L power:VCC #PWR?
+U 1 1 600700A3
+P 7650 4900
+F 0 "#PWR?" H 7650 4750 50  0001 C CNN
+F 1 "VCC" H 7665 5073 50  0000 C CNN
+F 2 "" H 7650 4900 50  0001 C CNN
+F 3 "" H 7650 4900 50  0001 C CNN
+	1    7650 4900
+	1    0    0    -1
+$EndComp
+Wire Wire Line
+	7650 4900 7650 5025
 $EndSCHEMATC

Commit message: 3
Parts:
- added Dioda1: DIODE, symbol Simulation_SPICE:DIODE
- added bzučák1: Buzzer, symbol Device:Buzzer
- Rec1, Rec2, Rec3: footprint (none) -> Resistor_SMD:R_0805_2012Metric
- renumbered Nastavení to Nastaven1
Connections:
- net GND: now also Dioda1.1 (A), bzučák1.2 (+)
- new net: Dioda1.2 (K), bzučák1.1 (-)
Other:
- note added: "Bzučák\n"
Changed lines of the file:
@@
 $EndComp
 $Comp
-L Device:Rotary_Encoder_Switch Nastavení
+L Device:Rotary_Encoder_Switch Nastaven1
 U 1 1 60004A19
 P 9125 5725
-F 0 "Nastavení" H 9125 6092 50  0000 C CNN
-F 1 "nastavení hodin" H 9125 6001 50  0000 C CNN
+F 0 "Nastaven1" H 9100 6200 50  0000 C CNN
+F 1 "nastavení hodin" H 9100 6125 50  0000 C CNN
 F 2 "" H 8975 5885 50  0001 C CNN
 F 3 "~" H 9125 5985 50  0001 C CNN
@@
 F 0 "Rec1" H 8545 5221 50  0000 L CNN
 F 1 "10K" H 8545 5130 50  0000 L CNN
-F 2 "" V 8405 5175 50  0001 C CNN
+F 2 "Resistor_SMD:R_0805_2012Metric" V 8405 5175 50  0001 C CNN
 F 3 "~" H 8475 5175 50  0001 C CNN
 	1    8475 5175
@@
 F 0 "Rec2" H 8245 5221 50  0000 L CNN
 F 1 "10K" H 8245 5130 50  0000 L CNN
-F 2 "" V 8105 5175 50  0001 C CNN
+F 2 "Resistor_SMD:R_0805_2012Metric" V 8105 5175 50  0001 C CNN
 F 3 "~" H 8175 5175 50  0001 C CNN
 	1    8175 5175
@@
 F 0 "Rec3" H 7945 5221 50  0000 L CNN
 F 1 "10K" H 7945 5130 50  0000 L CNN
-F 2 "" V 7805 5175 50  0001 C CNN
+F 2 "Resistor_SMD:R_0805_2012Metric" V 7805 5175 50  0001 C CNN
 F 3 "~" H 7875 5175 50  0001 C CNN
 	1    7875 5175
@@
 	8600 5725 8600 6075
 $Comp
-L power:GND #PWR?
+L power:GND #PWR05
 U 1 1 6004F39A
 P 8600 6075
-F 0 "#PWR?" H 8600 5825 50  0001 C CNN
+F 0 "#PWR05" H 8600 5825 50  0001 C CNN
 F 1 "GND" H 8605 5902 50  0000 C CNN
 F 2 "" H 8600 6075 50  0001 C CNN
@@
 	9575 5825 9575 6025
 $Comp
-L power:GND #PWR?
+L power:GND #PWR06
 U 1 1 60054E38
 P 9575 6025
-F 0 "#PWR?" H 9575 5775 50  0001 C CNN
+F 0 "#PWR06" H 9575 5775 50  0001 C CNN
 F 1 "GND" H 9580 5852 50  0000 C CNN
 F 2 "" H 9575 6025 50  0001 C CNN
@@
 Connection ~ 7875 5025
 $Comp
-L power:VCC #PWR?
+L power:VCC #PWR04
 U 1 1 600700A3
 P 7650 4900
-F 0 "#PWR?" H 7650 4750 50  0001 C CNN
+F 0 "#PWR04" H 7650 4750 50  0001 C CNN
 F 1 "VCC" H 7665 5073 50  0000 C CNN
 F 2 "" H 7650 4900 50  0001 C CNN
@@
 Wire Wire Line
 	7650 4900 7650 5025
+Text Notes 3800 4750 0    50   ~ 0
+Bzučák\n
+$Comp
+L Device:Buzzer bzučák1
+U 1 1 60078352
+P 4725 5150
+F 0 "bzučák1" H 4877 5179 50  0000 L CNN
+F 1 "Buzzer" H 4877 5088 50  0000 L CNN
+F 2 "" V 4700 5250 50  0001 C CNN
+F 3 "~" V 4700 5250 50  0001 C CNN
+	1    4725 5150
+	1    0    0    -1
+$EndComp
+$Comp
+L power:GND #PWR03
+U 1 1 6007EDA1
+P 4325 5450
+F 0 "#PWR03" H 4325 5200 50  0001 C CNN
+F 1 "GND" H 4330 5277 50  0000 C CNN
+F 2 "" H 4325 5450 50  0001 C CNN
+F 3 "" H 4325 5450 50  0001 C CNN
+	1    4325 5450
+	1    0    0    -1
+$EndComp
+$Comp
+L Simulation_SPICE:DIODE Dioda1
+U 1 1 60085D5E
+P 4325 5150
+F 0 "Dioda1" V 4371 5070 50  0000 R CNN
+F 1 "DIODE" V 4280 5070 50  0000 R CNN
+F 2 "" H 4325 5150 50  0001 C CNN
+F 3 "~" H 4325 5150 50  0001 C CNN
+F 4 "Y" H 4325 5150 50  0001 L CNN "Spice_Netlist_Enabled"
+F 5 "D" H 4325 5150 50  0001 L CNN "Spice_Primitive"
+	1    4325 5150
+	0    -1   -1   0
+$EndComp
+Wire Wire Line
+	4325 5300 4325 5350
+Wire Wire Line
+	4325 5350 4525 5350
+Wire Wire Line
+	4525 5350 4525 5250
+Wire Wire Line
+	4525 5250 4625 5250
+Connection ~ 4325 5350
+Wire Wire Line
+	4325 5350 4325 5450
+Wire Wire Line
+	4625 5050 4525 5050
+Wire Wire Line
+	4525 5050 4525 4925
+Wire Wire Line
+	4525 4925 4325 4925
+Wire Wire Line
+	4325 5000 4325 4925
+Connection ~ 4325 4925
+Wire Wire Line
+	4325 4925 4050 4925
 $EndSCHEMATC

Commit message: 3
Parts:
- Nastaven1: footprint (none) -> Rotary_Encoder:RotaryEncoder_Alps_EC11E-Switch_Vertical_H20mm
Changed lines of the file:
@@
 F 0 "Nastaven1" H 9100 6200 50  0000 C CNN
 F 1 "nastavení hodin" H 9100 6125 50  0000 C CNN
-F 2 "" H 8975 5885 50  0001 C CNN
+F 2 "Rotary_Encoder:RotaryEncoder_Alps_EC11E-Switch_Vertical_H20mm" H 8975 5885 50  0001 C CNN
 F 3 "~" H 9125 5985 50  0001 C CNN
 	1    9125 5725

Commit message: 10
Connections:
- net A: now reaches Nastaven1.A, Rec3.2
- net A: now also Digital1.3 (Pin_3)
- net B: now reaches Nastaven1.B, Rec2.2
- net B: now also Digital1.4 (Pin_4)
- net S1: now reaches Nastaven1.S1, Rec1.2
- net S1: now also Digital1.5 (Pin_5)
- net Buz: now reaches Dioda1.2 (K), bzučák1.1 (-)
- net Buz: now also Digital2.5 (Pin_5)
- no-connect marks 21 -> 20
Other:
- moved on the sheet: Dioda1, bzučák1
Changed lines of the file:
@@
 $EndComp
-Wire Notes Line
-	3850 7750 500  7750
 Wire Notes Line
 	400  5550 3750 5550
@@
 Y5
 Wire Notes Line
-	6975 4625 6975 6550
-Wire Notes Line
 	10900 6550 10900 4625
 Text Notes 10825 4975 2    118  ~ 0
@@
 A2
 NoConn ~ 2300 6800
-NoConn ~ 2050 3400
 NoConn ~ 2050 3300
 NoConn ~ 2050 3200
-NoConn ~ 2075 4600
-NoConn ~ 2075 4700
 NoConn ~ 2075 5100
 NoConn ~ 1025 4875
@@
 Wire Notes Line
 	3750 4625 10900 4625
-NoConn ~ 2075 4800
 NoConn ~ 2075 4900
 NoConn ~ 2075 5000
@@
 L Device:Buzzer bzučák1
 U 1 1 60078352
-P 4725 5150
-F 0 "bzučák1" H 4877 5179 50  0000 L CNN
-F 1 "Buzzer" H 4877 5088 50  0000 L CNN
-F 2 "" V 4700 5250 50  0001 C CNN
-F 3 "~" V 4700 5250 50  0001 C CNN
-	1    4725 5150
+P 5300 5150
+F 0 "bzučák1" H 5452 5179 50  0000 L CNN
+F 1 "Buzzer" H 5452 5088 50  0000 L CNN
+F 2 "" V 5275 5250 50  0001 C CNN
+F 3 "~" V 5275 5250 50  0001 C CNN
+	1    5300 5150
 	1    0    0    -1
 $EndComp
@@
 L power:GND #PWR03
 U 1 1 6007EDA1
-P 4325 5450
-F 0 "#PWR03" H 4325 5200 50  0001 C CNN
-F 1 "GND" H 4330 5277 50  0000 C CNN
-F 2 "" H 4325 5450 50  0001 C CNN
-F 3 "" H 4325 5450 50  0001 C CNN
-	1    4325 5450
+P 4900 5450
+F 0 "#PWR03" H 4900 5200 50  0001 C CNN
+F 1 "GND" H 4905 5277 50  0000 C CNN
+F 2 "" H 4900 5450 50  0001 C CNN
+F 3 "" H 4900 5450 50  0001 C CNN
+	1    4900 5450
 	1    0    0    -1
 $EndComp
@@
 L Simulation_SPICE:DIODE Dioda1
 U 1 1 60085D5E
-P 4325 5150
-F 0 "Dioda1" V 4371 5070 50  0000 R CNN
-F 1 "DIODE" V 4280 5070 50  0000 R CNN
-F 2 "" H 4325 5150 50  0001 C CNN
-F 3 "~" H 4325 5150 50  0001 C CNN
-F 4 "Y" H 4325 5150 50  0001 L CNN "Spice_Netlist_Enabled"
-F 5 "D" H 4325 5150 50  0001 L CNN "Spice_Primitive"
-	1    4325 5150
+P 4900 5150
+F 0 "Dioda1" V 4946 5070 50  0000 R CNN
+F 1 "DIODE" V 4855 5070 50  0000 R CNN
+F 2 "" H 4900 5150 50  0001 C CNN
+F 3 "~" H 4900 5150 50  0001 C CNN
+F 4 "Y" H 4900 5150 50  0001 L CNN "Spice_Netlist_Enabled"
+F 5 "D" H 4900 5150 50  0001 L CNN "Spice_Primitive"
+	1    4900 5150
 	0    -1   -1   0
 $EndComp
 Wire Wire Line
-	4325 5300 4325 5350
-Wire Wire Line
-	4325 5350 4525 5350
-Wire Wire Line
-	4525 5350 4525 5250
-Wire Wire Line
-	4525 5250 4625 5250
-Connection ~ 4325 5350
-Wire Wire Line
-	4325 5350 4325 5450
-Wire Wire Line
-	4625 5050 4525 5050
-Wire Wire Line
-	4525 5050 4525 4925
-Wire Wire Line
-	4525 4925 4325 4925
-Wire Wire Line
-	4325 5000 4325 4925
-Connection ~ 4325 4925
-Wire Wire Line
-	4325 4925 4050 4925
+	4900 5300 4900 5350
+Wire Wire Line
+	4900 5350 5100 5350
+Wire Wire Line
+	5100 5350 5100 5250
+Wire Wire Line
+	5100 5250 5200 5250
+Connection ~ 4900 5350
+Wire Wire Line
+	4900 5350 4900 5450
+Wire Wire Line
+	5200 5050 5100 5050
+Wire Wire Line
+	5100 5050 5100 4925
+Wire Wire Line
+	5100 4925 4900 4925
+Wire Wire Line
+	4900 5000 4900 4925
+Connection ~ 4900 4925
+Wire Wire Line
+	4900 4925 4625 4925
+Wire Notes Line
+	500  7750 6975 7750
+Wire Notes Line
+	6975 4625 6975 7750
+Text GLabel 4625 4925 0    39   Input ~ 0
+Buz
+Wire Wire Line
+	2050 3400 2250 3400
+Text GLabel 2250 3400 2    39   Input ~ 0
+Buz
+Wire Wire Line
+	2075 4600 2275 4600
+Text GLabel 2275 4600 2    39   Input ~ 0
+A
+Text GLabel 7725 5625 0    39   Input ~ 0
+A
+Text GLabel 7725 5825 0    39   Input ~ 0
+B
+Text GLabel 7725 5450 0    39   Input ~ 0
+S1
+Wire Wire Line
+	2075 4700 2275 4700
+Text GLabel 2275 4700 2    39   Input ~ 0
+B
+Wire Wire Line
+	2075 4800 2275 4800
+Text GLabel 2275 4800 2    39   Input ~ 0
+S1
+NoConn ~ 1025 4575
+NoConn ~ 1025 4475
+NoConn ~ 1025 4375
 $EndSCHEMATC

Commit message: 1
Parts:
- Dioda1: footprint (none) -> Diode_SMD:D_SMA
- bzučák1: footprint (none) -> Buzzer_Beeper:Buzzer_12x9.5RM7.6
Changed lines of the file:
@@
 F 0 "bzučák1" H 5452 5179 50  0000 L CNN
 F 1 "Buzzer" H 5452 5088 50  0000 L CNN
-F 2 "" V 5275 5250 50  0001 C CNN
+F 2 "Buzzer_Beeper:Buzzer_12x9.5RM7.6" V 5275 5250 50  0001 C CNN
 F 3 "~" V 5275 5250 50  0001 C CNN
 	1    5300 5150
@@
 F 0 "Dioda1" V 4946 5070 50  0000 R CNN
 F 1 "DIODE" V 4855 5070 50  0000 R CNN
-F 2 "" H 4900 5150 50  0001 C CNN
+F 2 "Diode_SMD:D_SMA" H 4900 5150 50  0001 C CNN
 F 3 "~" H 4900 5150 50  0001 C CNN
 F 4 "Y" H 4900 5150 50  0001 L CNN "Spice_Netlist_Enabled"

Commit message: start
Parts:
- removed Analogin1: Conn_01x06_Male, Connector_PinHeader_2.54mm:PinHeader_1x06_P2.54mm_Vertical, symbol Connector:Conn_01x06_Male
- removed I1, I3, I4, I5, I6, Inv1, Inv2, Inv21, Inv22: 74HC04, Package_SO:SO-14_3.9x8.65mm_P1.27mm, symbol 74xx:74HC04
- removed Power1: Conn_01x08_Male, Connector_PinHeader_2.54mm:PinHeader_1x08_P2.54mm_Vertical, symbol Connector:Conn_01x08_Male
- added A?: Arduino_UNO_R2, Module:Arduino_UNO_R2, symbol MCU_Module:Arduino_UNO_R2
- added unit 1 of U1
- added unit 2 of U1
- added unit 4 of U1
- added unit 5 of U1
- added unit 6 of U1
- added unit 7 of U1
- added U2: 74HC04, Package_SO:SO-16_3.9x9.9mm_P1.27mm, symbol 74xx:74HC04
- C1, C2: symbol Device:CP -> AP-rescue:CP-Device
- Nastaven1: symbol Device:Rotary_Encoder_Switch -> AP-rescue:Rotary_Encoder_Switch-Device
- U1: footprint Package_SO:SO-14_3.9x8.65mm_P1.27mm -> Package_SO:SO-16_3.9x9.9mm_P1.27mm
Connections:
- net A: now also A?.20 (D5); no longer Digital1.3 (Pin_3)
- net A0: now also A?.25 (D10); no longer Digital2.8 (Pin_8)
- net A1: now also A?.26 (D11); no longer Digital2.7 (Pin_7)
- net A2: now also A?.27 (D12); no longer Digital2.6 (Pin_6)
- net B: now also A?.19 (D4); no longer Digital1.4 (Pin_4)
- net Buz: now also A?.28 (D13); no longer Digital2.5 (Pin_5)
- net GND: now also A?.29 (GND), A?.6 (GND), A?.7 (GND), U1.7 (GND), U2.7 (GND)
- net GNDs12: now also A?.24 (D9); no longer Digital2.9 (Pin_9)
- net GNDs6: now also A?.21 (D6); no longer Digital1.2 (Pin_2)
- net GNDs8: now also A?.22 (D7); no longer Digital1.1 (Pin_1)
- net GNDs9: now also A?.23 (D8); no longer Digital2.10 (Pin_10)
- net S1: now also A?.18 (D3); no longer Digital1.5 (Pin_5)
- net SCL: now also A?.14 (SCL/A5); no longer Digital2.1 (Pin_1)
- net SDA: now also A?.13 (SDA/A4); no longer Digital2.2 (Pin_2)
- net VCC: now also A?.5 (+5V), U1.14 (VCC), U2.14 (VCC)
- net Y0: now also U1.1
- net Y1: now also U1.3
- net Y3: now also U1.9
- net Y4: now also U1.11
- net Y5: now also U1.13
- net Y6: now also U2.1
- net Y7: now also U2.3
- net at Displej1.1 (e): now also U1.10
- net at Displej1.10 (f): now also U1.12
- net at Displej1.11 (a): now also U1.2
- net at Displej1.2 (d): now also U1.8
- net at Displej1.3 (DPX): now also U2.4
- net at Displej1.5 (g): now also U2.2
- net at Displej1.7 (b): now also U1.4
- no-connect marks 20 -> 8
Other:
- moved on the sheet: Digital1, Digital2

Commit message: start2
Parts:
- removed Digital1: Conn_01x08_Male, Connector_PinHeader_2.54mm:PinHeader_1x08_P2.54mm_Vertical, symbol Connector:Conn_01x08_Male
- removed Digital2: Conn_01x10_Male, Connector_PinHeader_2.54mm:PinHeader_1x10_P2.54mm_Vertical, symbol Connector:Conn_01x10_Male
- gave numbers to parts that had none: 1
Connections:
- no-connect marks 8 -> 6
Changed lines of the file:
@@
 Text Notes 9375 700  0    118  ~ 0
 Invertory a 7seg\n
-$Comp
-L Connector:Conn_01x08_Male Digital1
-U 1 1 600E7476
-P 9100 4150
-F 0 "Digital1" H 9208 4631 50  0000 C CNN
-F 1 "Conn_01x08_Male" H 9208 4540 50  0000 C CNN
-F 2 "Connector_PinHeader_2.54mm:PinHeader_1x08_P2.54mm_Vertical" H 9100 4150 50  0001 C CNN
-F 3 "~" H 9100 4150 50  0001 C CNN
-	1    9100 4150
-	1    0    0    -1
-$EndComp
-$Comp
-L Connector:Conn_01x10_Male Digital2
-U 1 1 600E8C6F
-P 9075 2850
-F 0 "Digital2" H 9183 3431 50  0000 C CNN
-F 1 "Conn_01x10_Male" H 9183 3340 50  0000 C CNN
-F 2 "Connector_PinHeader_2.54mm:PinHeader_1x10_P2.54mm_Vertical" H 9075 2850 50  0001 C CNN
-F 3 "~" H 9075 2850 50  0001 C CNN
-	1    9075 2850
-	1    0    0    -1
-$EndComp
 Text Notes 2475 2675 0    118  ~ 0
 Piny procesor\n
@@
 A2
 NoConn ~ 2300 6800
-NoConn ~ 9275 2750
-NoConn ~ 9275 2650
 NoConn ~ 9300 4550
 Wire Notes Line
@@
 $EndComp
 $Comp
-L MCU_Module:Arduino_UNO_R2 A?
+L MCU_Module:Arduino_UNO_R2 A1
 U 1 1 6006856E
 P 2150 4000
-F 0 "A?" H 1525 5100 50  0000 C CNN
+F 0 "A1" H 1525 5100 50  0000 C CNN
 F 1 "Arduino_UNO_R2" H 1500 5025 50  0000 C CNN
 F 2 "Module:Arduino_UNO_R2" H 2150 4000 50  0001 C CIN
@@
 	2250 5200 2250 5100
 $Comp
-L power:VCC #PWR?
+L power:VCC #PWR0108
 U 1 1 601143F4
 P 2350 2900
-F 0 "#PWR?" H 2350 2750 50  0001 C CNN
+F 0 "#PWR0108" H 2350 2750 50  0001 C CNN
 F 1 "VCC" H 2365 3073 50  0000 C CNN
 F 2 "" H 2350 2900 50  0001 C CNN
