File: _autosave-AP.sch (KiCad schematic (older format))
At the start: 32 parts, among them U1 74HC04

Commit message: start
Parts:
- removed Analogin1: Conn_01x06_Male, Connector_PinHeader_2.54mm:PinHeader_1x06_P2.54mm_Vertical, symbol Connector:Conn_01x06_Male
- removed Digital1, Power1: Conn_01x08_Male, Connector_PinHeader_2.54mm:PinHeader_1x08_P2.54mm_Vertical, symbol Connector:Conn_01x08_Male
- removed Digital2: Conn_01x10_Male, Connector_PinHeader_2.54mm:PinHeader_1x10_P2.54mm_Vertical, symbol Connector:Conn_01x10_Male
- removed I1, I3, I4, I5, I6, Inv1, Inv2, Inv21, Inv22: 74HC04, Package_SO:SO-14_3.9x8.65mm_P1.27mm, symbol 74xx:74HC04
- added A1: Arduino_UNO_R2, Module:Arduino_UNO_R2, symbol MCU_Module:Arduino_UNO_R2
- added unit 1 of U1
- added unit 2 of U1
- added unit 4 of U1
- added unit 5 of U1
- added unit 6 of U1
- added unit 7 of U1
- added U2: 74HC04, Package_SO:SO-16_3.9x9.9mm_P1.27mm, symbol 74xx:74HC04
- C1, C2: symbol Device:CP -> AP-rescue:CP-Device
- Nastaven1: symbol Device:Rotary_Encoder_Switch -> AP-rescue:Rotary_Encoder_Switch-Device
- U1: footprint Package_SO:SO-14_3.9x8.65mm_P1.27mm -> Package_SO:SO-16_3.9x9.9mm_P1.27mm
Connections:
- net A: now also A1.20 (D5)
- net A0: now also A1.25 (D10)
- net A1: now also A1.26 (D11)
- net A2: now also A1.27 (D12)
- net B: now also A1.19 (D4)
- net Buz: now also A1.28 (D13)
- net GND: now also A1.29 (GND), A1.6 (GND), A1.7 (GND), U1.7 (GND), U2.7 (GND)
- net GNDs12: now also A1.24 (D9)
- net GNDs6: now also A1.21 (D6)
- net GNDs8: now also A1.22 (D7)
- net GNDs9: now also A1.23 (D8)
- net S1: now also A1.18 (D3)
- net SCL: now also A1.14 (SCL/A5)
- net SDA: now also A1.13 (SDA/A4)
- net VCC: now also A1.5 (+5V), U1.14 (VCC), U2.14 (VCC)
- net Y0: now also U1.1
- net Y1: now also U1.3
- net Y3: now also U1.9
- net Y4: now also U1.11
- net Y5: now also U1.13
- net Y6: now also U2.1
- net Y7: now also U2.3
- net at Displej1.1 (e): now also U1.10
- net at Displej1.10 (f): now also U1.12
- net at Displej1.11 (a): now also U1.2
- net at Displej1.2 (d): now also U1.8
- net at Displej1.3 (DPX): now also U2.4
- net at Displej1.5 (g): now also U2.2
- net at Displej1.7 (b): now also U1.4
- no-connect marks 20 -> 6
