File: AP.kicad_pcb (KiCad board)
At the start: 2 copper layers, 16 parts, among them J1 Conn_01x06_Female, J2 Conn_01x01_Female, J3 Conn_01x02_Female, J4 Conn_01x03_Female, J5 Conn_01x01_Female, J6 Conn_01x04_Female, U1 74HC04, U2 DS3231MZ, U3 74HC04, U4 74HC04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

Commit message: 1
Parts:
- removed J1: Conn_01x06_Female, Connector_PinHeader_2.54mm:PinHeader_1x06_P2.54mm_Vertical
- removed J2, J5: Conn_01x01_Female, Connector_PinHeader_2.54mm:PinHeader_1x01_P2.54mm_Vertical
- removed J3: Conn_01x02_Female, Connector_PinHeader_2.54mm:PinHeader_1x02_P2.54mm_Vertical
- removed J4: Conn_01x03_Female, Connector_PinHeader_2.54mm:PinHeader_1x03_P2.54mm_Vertical
- removed J6: Conn_01x04_Female, Connector_PinHeader_2.54mm:PinHeader_1x04_P2.54mm_Vertical
- removed R1: RTRIM, Potentiometer_THT:Potentiometer_ACP_CA6-H2,5_Horizontal
- removed R2, R3, R4, R5: R, Resistor_THT:R_Axial_DIN0204_L3.6mm_D1.6mm_P5.08mm_Horizontal
- removed U1, U3: 74HC04, Package_DIP:DIP-14_W7.62mm_Socket
- removed U2: DS3231MZ, Connector_PinHeader_2.54mm:PinHeader_1x06_P2.54mm_Vertical
- removed U4: 74HC04, Package_DIP:DIP-16_W7.62mm
- removed U5: 74HC04, Display_7Segment:CA56-12SRWA
Routing:
- net VCC: track 195.6 -> 0.00 mm
- net Net-(U3-Pad1): track 93.0 -> 0.00 mm
- net Net-(U1-Pad3): track 74.9 -> 0.00 mm
- net Net-(U1-Pad1): track 52.1 -> 0.00 mm
- net Net-(R5-Pad2): track 20.3 -> 0.00 mm
- net Net-(J3-Pad2): track 17.8 -> 0.00 mm
- net Net-(J3-Pad1): track 17.8 -> 0.00 mm
- net Net-(J6-Pad4): track 14.0 -> 0.00 mm
- net Net-(J6-Pad3): track 12.7 -> 0.00 mm
- net Net-(U3-Pad4): track 11.4 -> 0.00 mm
- net Net-(U3-Pad2): track 11.4 -> 0.00 mm
- net Net-(J6-Pad2): track 11.4 -> 0.00 mm
- net Net-(J6-Pad1): track 8.89 -> 0.00 mm
- net Net-(J4-Pad1): track 6.88 -> 0.00 mm
- net Net-(R2-Pad2): track 5.08 -> 0.00 mm
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- removed copper zone on F.Cu, net GND

Commit message: start
Parts:
- added A1: Arduino_UNO_R2, Module:Arduino_UNO_R2, F.Cu at (162.0, 72.5)
- added Baterie1: Battery_Cell, Battery:BatteryHolder_Keystone_1060_1x2032, B.Cu at (182.4, 106.9)
- added C1: 10nF, Capacitor_SMD:C_0805_2012Metric, F.Cu at (19.8, 52.9)
- added C2: 1nF, Capacitor_SMD:C_0805_2012Metric, F.Cu at (37.2, 45.9)
- added Demultiplexor1: 74HC138, Package_SO:SO-16_3.9x9.9mm_P1.27mm, B.Cu at (193.5, 88.6)
- added Dioda1: DIODE, Diode_SMD:D_SMA, F.Cu at (13.5, 53.6)
- added Displej1: Disp, Display_7Segment:CA56-12SRWA, F.Cu at (166.1, 100.8)
- added Nastaven1: nastavení hodin, Rotary_Encoder:RotaryEncoder_Alps_EC11E-Switch_Vertical_H20mm, F.Cu at (154.9, 85.1)
- added R1: 220, Resistor_SMD:R_0805_2012Metric, F.Cu at (24.2, 52.8)
- added R2: 220, Resistor_SMD:R_0805_2012Metric, F.Cu at (60.4, 23.4)
- added R3: 220, Resistor_SMD:R_0805_2012Metric, F.Cu at (60.4, 26.4)
- added R4: 220, Resistor_SMD:R_0805_2012Metric, F.Cu at (60.4, 29.3)
- added RI2c1: 4k7, Resistor_SMD:R_0805_2012Metric, F.Cu at (46.5, 54.8)
- added RI2c2: 4k7, Resistor_SMD:R_0805_2012Metric, F.Cu at (83.4, 21.4)
- added RTC1: DS3231MZ, Package_SO:SO-8_3.9x4.9mm_P1.27mm, B.Cu at (149.9, 107.7)
- added Rec1: 10K, Resistor_SMD:R_0805_2012Metric, F.Cu at (46.5, 48.9)
- added Rec2: 10K, Resistor_SMD:R_0805_2012Metric, F.Cu at (50.9, 48.9)
- added Rec3: 10K, Resistor_SMD:R_0805_2012Metric, F.Cu at (46.5, 51.8)
- added U1: 74HC04, Package_SO:SO-16_3.9x9.9mm_P1.27mm, B.Cu at (138.9, 90.7)
- added U2: 74HC04, Package_SO:SO-16_3.9x9.9mm_P1.27mm, B.Cu at (148.8, 90.9)
- added bzučák1: Buzzer, Buzzer_Beeper:Buzzer_12x9.5RM7.6, F.Cu at (176.8, 87.1)
Routing:
- added copper zone on B.Cu, net GND
- added copper zone on F.Cu, net GND
Other:
- board outline added: 71 x 54 mm

Commit message: 1
Parts:
- moved Dioda1 149.1 mm to (148.0, 118.1), turned to 270 degrees
- moved C1 146.1 mm to (156.1, 105.5), turned to 270 degrees
- moved R1 143.7 mm to (156.1, 109.9), turned to 270 degrees
- moved R2 120.0 mm to (148.7, 104.7)
- moved R3 120.0 mm to (148.7, 107.7)
- moved R4 120.0 mm to (148.7, 110.6)
- moved C2 119.2 mm to (143.5, 99.7)
- moved Rec2 109.6 mm to (148.0, 99.7)
- moved Rec1 108.4 mm to (151.3, 76.8)
- moved Rec3 108.4 mm to (151.3, 79.8)
- moved RI2c1 106.2 mm to (151.1, 73.0)
- moved RI2c2 95.5 mm to (160.7, 77.5)
- moved U1 46.6 mm to (185.4, 87.6), turned to 180 degrees
- moved RTC1 33.6 mm to (168.9, 80.0)
- moved U2 8.54 mm to (140.3, 90.2)
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
Commit message: 1
Parts:
- C1, C2, Dioda1, R1, R2, R3, R4, RI2c1, RI2c2, Rec1, Rec2, Rec3: moved to B.Cu
- moved RI2c1 6.87 mm to (150.8, 79.9)
- moved R2 6.83 mm to (147.6, 111.4)
- moved Rec3 6.65 mm to (150.9, 73.1)
- moved R1 5.59 mm to (156.1, 104.3), turned to 90 degrees
- moved R4 5.17 mm to (147.6, 105.5)
- moved C1 3.27 mm to (156.1, 108.8), turned to 90 degrees
- moved C2 3.17 mm to (141.0, 97.8), turned to 90 degrees
- moved Rec2 3.05 mm to (145.0, 98.8)
- moved R3 1.38 mm to (147.6, 108.5)
- moved U1 1.04 mm to (186.3, 87.0)
- moved Rec1 0.82 mm to (150.9, 76.1)
- moved A1 0.61 mm to (162.1, 72.6)
- moved Demultiplexor1 0.57 mm to (195.7, 86.7)
- turned Dioda1 to 90 degrees
Routing:
- net VCC: track 0.00 -> 140.5 mm, vias 0 -> 4
- net Y6: track 0.00 -> 108.3 mm, vias 0 -> 6
- net Y7: track 0.00 -> 101.0 mm, vias 0 -> 2
- net A: track 0.00 -> 78.1 mm, vias 0 -> 5
- net S1: track 0.00 -> 66.3 mm, vias 0 -> 5
- net B: track 0.00 -> 60.9 mm, vias 0 -> 4
- net GNDs6: track 0.00 -> 57.7 mm
- net Net-(Displej1-Pad7): track 0.00 -> 55.8 mm, vias 0 -> 2
- net A0: track 0.00 -> 54.8 mm, vias 0 -> 4
- net Net-(Displej1-Pad11): track 0.00 -> 54.8 mm, vias 0 -> 10
- net A2: track 0.00 -> 54.2 mm, vias 0 -> 2
- net A1: track 0.00 -> 53.2 mm, vias 0 -> 2
- net SCL: track 0.00 -> 52.6 mm, vias 0 -> 2
- net Buz: track 0.00 -> 49.9 mm
- net GNDs8: track 0.00 -> 49.3 mm
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