File: AP.kicad_pcb (KiCad board)
At the start: 2 copper layers, 71 x 54 mm, 21 parts, among them U1 74HC04, U2 74HC04

Commit message: finále
Parts:
- Displej1: value Disp -> Displej
Other:
- board text added: "Projekt: Digitální hodiny Tvůrci: Jaroslav Žížala Matěj Kraus Apsolventský projekt"

Commit message: posledni_oprava
Routing:
- net Net-(Displej1-Pad10): track 49.1 -> 49.7 mm
- net GND: vias 18 -> 24
