File: AP.kicad_pcb (KiCad board)
At the start: 2 copper layers, 71 x 54 mm, 21 parts, among them U1 74HC04, U2 74HC04

Commit message: 1
1
Parts:
- removed A1: Arduino_UNO_R2, Module:Arduino_UNO_R2
- Displej1: value Displej -> Disp
- U1, U2: footprint Package_SO:SO-16_3.9x9.9mm_P1.27mm -> Package_SO:SO-14_3.9x8.65mm_P1.27mm
- moved U1 0.74 mm to (185.9, 86.4)
Connections:
- RTC1 pad 1: (no net) -> Net-(RTC1-Pad1)
- RTC1 pad 3: (no net) -> Net-(RTC1-Pad3)
- RTC1 pad 4: (no net) -> Net-(RTC1-Pad4)
Routing:
- net GND: track 0.00 -> 6.02 mm
- net Y5: track 29.4 -> 34.7 mm, vias 2 -> 4
- net Y3: track 18.1 -> 22.8 mm
- net Net-(Displej1-Pad10): track 49.7 -> 53.9 mm
- net Y4: track 34.2 -> 38.2 mm, vias 8 -> 4
- net Net-(Displej1-Pad2): track 34.3 -> 37.2 mm, vias 4 -> 6
- net VCC: track 140.5 -> 137.7 mm
- net Net-(Displej1-Pad1): track 27.0 -> 29.1 mm
- net Net-(Displej1-Pad5): track 31.2 -> 32.1 mm
- net Y6: track 108.3 -> 109.0 mm
